Commit message: [MILESTONE] Endeffector appears on the robot in rviz but needs debugging as moveit does not work with it

File: src/endeffector_description/urdf/ur_with_endeffector.xacro (robot description, xacro)
@@ -1,9 +1,12 @@
 <?xml version="1.0"?>
 <robot name="ur_with_endeffector" xmlns:xacro="http://www.ros.org/wiki/xacro">
+  <xacro:arg name="ur_type" default="ur5e" />
+  <xacro:arg name="prefix" default="end_effector_" />
   <xacro:include filename="$(find ur_description)/urdf/ur.urdf.xacro" />
   <xacro:include filename="$(find endeffector_description)/urdf/endeffector.xacro" />
   <joint name="tool0_to_endeffector_base" type="fixed">
-    <parent link="tool0" />
-    <child link="base_link" /> <origin xyz="0 0 0" rpy="0 0 0" />
+    <parent link="tool0"/>
+    <child link="$(arg prefix)base_link"/>
+    <origin xyz="0 0 0" rpy="0 0 0" />
   </joint>
 </robot>

Commit message: [DEBUG] Adjust joint origin for tool0 to endeffector base

File: src/endeffector_description/urdf/ur_with_endeffector.xacro (robot description, xacro)
@@ -8,5 +8,5 @@
     <parent link="tool0"/>
     <child link="$(arg prefix)base_link"/>
-    <origin xyz="0 0 0" rpy="0 0 0" />
+    <origin xyz="0 0 0.08" rpy="0 0 3.14159" />
   </joint>
 </robot>
