Commit message: [DEBUG] Commit before main

File: src/endeffector_description/urdf/old/endeffector.xacro (robot description, xacro)
@@ -14,5 +14,5 @@
       <origin xyz="0 0 0" rpy="0 0 0"/>
       <geometry>
-        <mesh filename="package://endeffector_description/meshes/base_link.stl" scale="0.001 0.001 0.001"/>
+        <mesh filename="file://$(find endeffector_description)/meshes/base_link.stl" scale="0.001 0.001 0.001"/>
       </geometry>
       <material name="silver"/>
@@ -22,16 +22,9 @@
       <origin xyz="0 0 0" rpy="0 0 0"/>
       <geometry>
-        <mesh filename="package://endeffector_description/meshes/base_link.stl" scale="0.001 0.001 0.001"/>
+        <mesh filename="file://$(find endeffector_description)/meshes/base_link.stl" scale="0.001 0.001 0.001"/>
       </geometry>
     </collision>
     -->
-    <!-- inserted by tool: default collision -->
-    <collision>
-      <geometry>
-        <box size="0.06 0.04 0.03"/>
-      </geometry>
-      <origin xyz="0 0 0.015" rpy="0 0 0"/>
-    </collision>
-</link>
+  </link>
   <link name="$(arg prefix)Component3_1">
     <inertial>
@@ -43,5 +36,5 @@
       <origin xyz="-0.000468 0.003253 -0.016" rpy="0 0 0"/>
       <geometry>
-        <mesh filename="package://endeffector_description/meshes/Component3_1.stl" scale="0.001 0.001 0.001"/>
+        <mesh filename="file://$(find endeffector_description)/meshes/Component3_1.stl" scale="0.001 0.001 0.001"/>
       </geometry>
       <material name="silver"/>
@@ -51,16 +44,9 @@
       <origin xyz="-0.000468 0.003253 -0.016" rpy="0 0 0"/>
       <geometry>
-        <mesh filename="package://endeffector_description/meshes/Component3_1.stl" scale="0.001 0.001 0.001"/>
+        <mesh filename="file://$(find endeffector_description)/meshes/Component3_1.stl" scale="0.001 0.001 0.001"/>
       </geometry>
     </collision>
     -->
-    <!-- inserted by tool: default collision -->
-    <collision>
-      <geometry>
-        <box size="0.06 0.04 0.03"/>
-      </geometry>
-      <origin xyz="0 0 0.015" rpy="0 0 0"/>
-    </collision>
-</link>
+  </link>
   <link name="$(arg prefix)Capacative_Soil_Moisture_Sensor_v1.2_v2_1">
     <inertial>
@@ -72,5 +58,5 @@
       <origin xyz="0.010632 0.094013 -0.02415" rpy="0 0 0"/>
       <geometry>
-        <mesh filename="package://endeffector_description/meshes/Capacative_Soil_Moisture_Sensor_v1.2_v2_1.stl" scale="0.001 0.001 0.001"/>
+        <mesh filename="file://$(find endeffector_description)/meshes/Capacative_Soil_Moisture_Sensor_v1.2_v2_1.stl" scale="0.001 0.001 0.001"/>
       </geometry>
       <material name="silver"/>
@@ -80,16 +66,9 @@
       <origin xyz="0.010632 0.094013 -0.02415" rpy="0 0 0"/>
       <geometry>
-        <mesh filename="package://endeffector_description/meshes/Capacative_Soil_Moisture_Sensor_v1.2_v2_1.stl" scale="0.001 0.001 0.001"/>
+        <mesh filename="file://$(find endeffector_description)/meshes/Capacative_Soil_Moisture_Sensor_v1.2_v2_1.stl" scale="0.001 0.001 0.001"/>
       </geometry>
     </collision>
     -->
-    <!-- inserted by tool: default collision -->
-    <collision>
-      <geometry>
-        <box size="0.06 0.04 0.03"/>
-      </geometry>
-      <origin xyz="0 0 0.015" rpy="0 0 0"/>
-    </collision>
-</link>
+  </link>
   <joint name="$(arg prefix)Rigid 2" type="fixed">
     <origin xyz="0.000468 -0.003253 0.016" rpy="0 0 0"/>

File: src/endeffector_description/urdf/ur_with_endeffector.xacro (robot description, xacro)
@@ -1,13 +1,34 @@
 <?xml version="1.0"?>
 <robot name="ur_with_endeffector" xmlns:xacro="http://www.ros.org/wiki/xacro">
-  <xacro:arg name="name" default="ur5" />
-  <xacro:arg name="ur_type" default="ur5" />
-  <xacro:arg name="prefix" default="end_effector_" />
+  <xacro:arg name="name" default="ur5e" />
+  <xacro:arg name="ur_type" default="ur5e" />
   <xacro:include filename="$(find ur_description)/urdf/ur.urdf.xacro" />
-  <xacro:include filename="$(find endeffector_description)/urdf/endeffector.xacro" />
+  <link name="simple_ee_link">
+    <visual>
+      <geometry>
+        <box size="0.05 0.05 0.15"/>  <!-- Length, Width, Height -->
+      </geometry>
+      <material name="orange">
+        <color rgba="1.0 0.5 0.0 1.0"/>
+      </material>
+    </visual>
+    <collision>
+      <geometry>
+        <box size="0.05 0.05 0.15"/>  <!-- Must match visual -->
+      </geometry>
+    </collision>
+    <inertial>
+    <mass value="2.0"/>  <!-- 2kg mass -->
+    <!-- Calculated inertia for a rectangular prism -->
+    <inertia
+      ixx="0.01625" ixy="0.0" ixz="0.0"
+      iyy="0.0085" iyz="0.0"
+      izz="0.00425"/>
+  </inertial>
+  </link>
   <joint name="tool0_to_endeffector_base" type="fixed">
     <parent link="tool0"/>
-    <child link="$(arg prefix)base_link"/>
-    <origin xyz="0 0 0.08" rpy="0 0 3.14159" />
+    <child link="simple_ee_link"/>
+    <origin xyz="0 0 0.08" rpy="0 0 0" />
   </joint>
 </robot>
